File: PCB/Mainboard/Mainboard/Mainboard.sch (EAGLE design)
At the start: 18 parts

Commit message: Added missing leg controller +  layout
Parts:
- added BUTTON1, BUTTON2, BUTTON3, BUTTON4, BUTTON5: (no value), pinhead:PINHD-1X2
- added C3, C4, C5, C6, C7: (no value), rcl:C-EUC0805
- added LED10, LED11, LED12, LED3, LED4, LED5, LED6, LED7, LED8, LED9: (no value), led:LEDCHIP-LED0805
- added LEG2, LEG3, LEG4, LEG5, LEG6: ATTINY1614, ATTINY1614:ATTINY1614/16/17SSNR/SSFR
- added R10, R11, R12, R3, R4, R5, R6, R7, R8, R9: (no value), rcl:R-EU_R0805
- added SERVO10, SERVO11, SERVO12, SERVO13, SERVO14, SERVO15, SERVO16, SERVO17, SERVO18, SERVO4, SERVO5, SERVO6, SERVO7, SERVO8, SERVO9: (no value), pinhead:PINHD-1X3
- added SJ10, SJ11, SJ12, SJ13, SJ14, SJ15, SJ16, SJ17, SJ18, SJ4, SJ5, SJ6, SJ7, SJ8, SJ9: (no value), jumper:SJ
Connections:
- net ADDR0 renamed N$3
- net ADDR1 renamed N$4
- net ADDR2 renamed N$5
- net BTN renamed N$8
- net LED1 renamed N$1
- net LED2 renamed N$2
- net S1 renamed N$9
- net S2 renamed N$10
- net S3 renamed N$12
- removed net N$16: JP6.5
- removed net N$17: JP6.7
- removed net N$18: JP6.2
- removed net N$19: JP6.4
- removed net N$20: JP6.6
- removed net N$21: JP6.8
- new net N$11: LED3.A, R3.2
- new net N$13: LED4.A, R4.2
- new net N$14: LEG2.PB2(TXD), R3.1
- new net N$15: LEG2.PB3(RXD), R4.1
- new net N$22: LEG2.PA1(MOSI), SJ4.1
- new net N$23: LEG2.PA2(MISO), SJ5.1
- new net N$24: LEG2.PA3(SCK), SJ6.1
- new net N$25: BUTTON1.1, LEG2.PA4(!SS!)
- new net N$26: LEG2.PA5, SERVO4.1
- new net N$27: LEG2.PA6, SERVO5.1
- new net N$28: LEG2.PA7, SERVO6.1
- new net N$29: LED5.A, R5.2
- new net N$30: LED6.A, R6.2
- new net N$31: LEG3.PB2(TXD), R5.1
- new net N$32: LEG3.PB3(RXD), R6.1
- new net N$33: LEG3.PA1(MOSI), SJ7.1
- new net N$34: LEG3.PA2(MISO), SJ8.1
- new net N$35: LEG3.PA3(SCK), SJ9.1
- new net N$36: BUTTON2.1, LEG3.PA4(!SS!)
- new net N$37: LEG3.PA5, SERVO7.1
- new net N$38: LEG3.PA6, SERVO8.1
- new net N$39: LEG3.PA7, SERVO9.1
- new net N$40: LED7.A, R7.2
- new net N$41: LED8.A, R8.2
- new net N$42: LEG4.PB2(TXD), R7.1
- new net N$43: LEG4.PB3(RXD), R8.1
- new net N$44: LEG4.PA1(MOSI), SJ10.1
- new net N$45: LEG4.PA2(MISO), SJ11.1
- new net N$46: LEG4.PA3(SCK), SJ12.1
- new net N$47: BUTTON3.1, LEG4.PA4(!SS!)
- new net N$48: LEG4.PA5, SERVO10.1
- new net N$49: LEG4.PA6, SERVO11.1
- new net N$50: LEG4.PA7, SERVO12.1
- new net N$51: LED9.A, R9.2
- new net N$52: LED10.A, R10.2
- new net N$53: LEG5.PB2(TXD), R9.1
- new net N$54: LEG5.PB3(RXD), R10.1
- new net N$55: LEG5.PA1(MOSI), SJ13.1
- new net N$56: LEG5.PA2(MISO), SJ14.1
- new net N$57: LEG5.PA3(SCK), SJ15.1
- new net N$58: BUTTON4.1, LEG5.PA4(!SS!)
- new net N$59: LEG5.PA5, SERVO13.1
- new net N$60: LEG5.PA6, SERVO14.1
- new net N$61: LEG5.PA7, SERVO15.1
- new net N$62: LED11.A, R11.2
- new net N$63: LED12.A, R12.2
- new net N$64: LEG6.PB2(TXD), R11.1
- new net N$65: LEG6.PB3(RXD), R12.1
- new net N$66: LEG6.PA1(MOSI), SJ16.1
- new net N$67: LEG6.PA2(MISO), SJ17.1
- new net N$68: LEG6.PA3(SCK), SJ18.1
- new net N$69: BUTTON5.1, LEG6.PA4(!SS!)
- new net N$70: LEG6.PA5, SERVO16.1
- new net N$71: LEG6.PA6, SERVO17.1
- new net N$72: LEG6.PA7, SERVO18.1
- new net UPDI2: JP6.5, LEG2.PA0(!RST!/UPDI/A0)
- new net UPDI3: JP6.7, LEG3.PA0(!RST!/UPDI/A0)
- new net UPDI4: JP6.4, LEG4.PA0(!RST!/UPDI/A0)
- new net UPDI5: JP6.6, LEG5.PA0(!RST!/UPDI/A0)
- new net UPDI6: JP6.8, LEG6.PA0(!RST!/UPDI/A0)
- new net VCC/2: SERVO10.2, SERVO11.2, SERVO12.2, SERVO13.2, SERVO14.2, SERVO15.2, SERVO16.2, SERVO17.2, SERVO18.2
- net +5V: now also C3.1, C4.1, C5.1, C6.1, C7.1, LEG2.VCC, LEG3.VCC, LEG4.VCC, LEG5.VCC, LEG6.VCC
- net GND: now also BUTTON1.2, BUTTON2.2, BUTTON3.2, BUTTON4.2, BUTTON5.2, C3.2, C4.2, C5.2, C6.2, C7.2, JP6.2, LED10.C, LED11.C, LED12.C, LED3.C, LED4.C, LED5.C, LED6.C, LED7.C, LED8.C, LED9.C, LEG2.GND, LEG3.GND, LEG4.GND, LEG5.GND, LEG6.GND, SERVO10.3, SERVO11.3, SERVO12.3, SERVO13.3, SERVO14.3, SERVO15.3, SERVO16.3, SERVO17.3, SERVO18.3, SERVO4.3, SERVO5.3, SERVO6.3, SERVO7.3, SERVO8.3, SERVO9.3, SJ10.2, SJ11.2, SJ12.2, SJ13.2, SJ14.2, SJ15.2, SJ16.2, SJ17.2, SJ18.2, SJ4.2, SJ5.2, SJ6.2, SJ7.2, SJ8.2, SJ9.2
- net SCL: now also LEG2.PB0(SCL), LEG3.PB0(SCL), LEG4.PB0(SCL), LEG5.PB0(SCL), LEG6.PB0(SCL)
- net SDA: now also LEG2.PB1(SDA), LEG3.PB1(SDA), LEG4.PB1(SDA), LEG5.PB1(SDA), LEG6.PB1(SDA)
- net VCC: now also SERVO4.2, SERVO5.2, SERVO6.2, SERVO7.2, SERVO8.2, SERVO9.2

Commit message: Finished layout for current circuit
Parts:
- added R13, R14: (no value), rcl:R-EU_R0805
- SJ1, SJ10, SJ11, SJ12, SJ13, SJ14, SJ15, SJ16, SJ17, SJ18, SJ2, SJ3, SJ4, SJ5, SJ6, SJ7, SJ8, SJ9: device jumper:SJ -> rcl:R-EU_R0402
Connections:
- net +5V: now also R13.2, R14.2
- net SCL: now also R14.1
- net SDA: now also R13.1
- net UPDI0: now also JP6.6; no longer JP6.1
- net UPDI1: now also JP6.5; no longer JP6.3
- net UPDI2: now also JP6.8; no longer JP6.5
- net UPDI5: now also JP6.3; no longer JP6.6
- net UPDI6: now also JP6.1; no longer JP6.8
Other:
- note added: "TODO: Sensor I2C-Port 3.3V Regler 5V Regler? Power-Verbinder Led? Buttoncon?"
