File: PCB/Mainboard/Mainboard.sch (EAGLE design)
At the start: 25 parts, among them IC1 FT232RL

Commit message: added new parts, added all signals
Parts:
- removed U$100: ESP32-DOITV1, HeRo:ESP32-DOITV1
- added C3: 100nF, rcl:C-EUC0805
- added C4, C5, C6: 1nF, rcl:C-EUC0805
- added LED3, LED4, LED5, LED6, LED7: (no value), led:LEDCHIP-LED0805
- added R10, R12, R9: 1k, rcl:R-EU_R0805
- added R11, R22, R23, R24, R25, R7, R8: 10k, rcl:R-EU_R0805
- added R13, R14: 470R, rcl:R-EU_R0805
- added R15, R16, R17, R18, R21: (no value), rcl:R-EU_R0805
- added R19, R20, R27, R28: 0R, rcl:R-EU_R0805
- added R26: 200k, rcl:R-EU_R0805
- added S1, S2: (no value), switch-omron:10-XX
- added S3, S4, S5: (no value), switch:255SB
- added SJ1: (no value), jumper:SJ
- added T1, T2: BC847, transistor:BC847
- added U$2: ESP32-WROOM-32U, HeRo:ESP32-WROOM-32U
- added U$5: BLUEDOT-BNO055, HeRo:BLUEDOT-BNO055
- added U$6: D24V10F3, HeRo:D24V10F3
- added U$7: PCA9306, HeRo:PCA9306
Connections:
- removed net N$1: C1.1, IC1.3V3OUT, IC1.VCCIO, R4.1, R5.2, R6.2
- removed net SCL: LEG1.5, LEG2.5, LEG3.5, LEG4.5, LEG5.5, LEG6.5
- removed net SDA: LEG1.6, LEG2.6, LEG3.6, LEG4.6, LEG5.6, LEG6.6
- new net CLK: U$2.CLK
- new net CMD: U$2.CMD
- new net EN: C4.1, R11.1, R13.1, T1.C, U$2.EN
- new net EN_3V3: S5.P, U$6.!SHDN
- new net IMU_ADR: SJ1.1, U$5.ADR
- new net IMU_INT: R21.1, U$5.INT
- new net IO0: R14.1, T2.C, U$2.IO0
- new net IO12: U$2.IO12
- new net IO13: U$2.IO13
- new net IO14: U$2.IO14
- new net IO15: U$2.IO15
- new net IO16: U$2.IO16
- new net IO17: R21.2, U$2.IO17
- new net IO18: R19.1, U$2.IO18
- new net IO19: R20.1, U$2.IO19
- new net IO2: R12.2, U$2.IO2
- new net IO21: U$2.IO21
- new net IO22: R27.1, U$2.IO22
- new net IO23: R28.1, U$2.IO23
- new net IO25: U$2.IO25
- new net IO26: U$2.IO26
- new net IO27: U$2.IO27
- new net IO32: U$2.IO32
- new net IO33: U$2.IO33
- new net IO34: U$2.IO34
- new net IO35: U$2.IO35
- new net IO4: U$2.IO4
- new net IO5: U$2.IO5
- new net N$12: LED3.A, R12.1
- new net N$13: C5.1, R13.2, S1.S, S1.S1
- new net N$14: C6.1, R14.2, S2.S, S2.S1
- new net N$15: LED5.A, R16.1
- new net N$16: LED6.A, R17.1
- new net N$17: LED4.A, R15.1
- new net N$18: LED7.A, R18.1
- new net N$23: R26.2, U$7.EN, U$7.VREF2
- new net N$8: R7.1, T1.B
- new net N$9: R8.1, T2.B
- new net RXD0: R9.2, U$2.RXD0
- new net SCL_3V3: R22.2, R27.2, U$7.SCL1
- new net SD0: U$2.SD0
- new net SD1: U$2.SD1
- new net SD2: U$2.SD2
- new net SD3: U$2.SD3
- new net SDA_3V3: R23.2, R28.2, U$7.SDA1
- new net SN: U$2.SENSOR_VN
- new net SP: U$2.SENSOR_VP
- new net TXD0: R10.2, U$2.TXD0
- net !DTR: now also R7.2, T2.E
- net !RTS: now also R8.2, T1.E
- net +12V: now also R18.2, U$6.VIN
- net +3V3: now also C1.1, C3.1, IC1.VCCIO, R11.2, R15.2, R22.1, R23.1, R4.1, R5.2, R6.2, U$2.3V3, U$6.VOUT, U$7.VREF1
- net +5V: now also R16.2, R24.1, R25.1, R26.1, U$5.VCC
- net EN_5V: now also S4.P
- net EN_SERVO: now also S3.P
- net GND: now also C3.2, C4.2, C5.2, C6.2, LED3.C, LED4.C, LED5.C, LED6.C, LED7.C, S1.P, S1.P1, S2.P, S2.P1, S3.S, S4.S, S5.S, SJ1.2, U$2.GND, U$5.GND, U$6.GND, U$7.GND
- net PG_LEG: now also R19.2
- net PG_SERVO: now also R20.2
- net RXD: now also R10.1
- net SCL_5V: now also LEG1.5, LEG2.5, LEG3.5, LEG4.5, LEG5.5, LEG6.5, R24.2, U$5.SCL, U$7.SCL2
- net SDA_5V: now also LEG1.6, LEG2.6, LEG3.6, LEG4.6, LEG5.6, LEG6.6, R25.2, U$5.SDA, U$7.SDA2
- net TXD: now also R9.1
- net VDD: now also R17.2

Commit message: minor adjustments, finished routing
Parts:
- removed R19, R20: 0R, rcl:R-EU_R0805
- removed R2, R3: 10k, rcl:R-EU_R0805
- removed R21: (no value), rcl:R-EU_R0805
- removed S1, S2: (no value), switch-omron:10-XX
- removed U$1: VL53L0XV, HeRo:VL53L0XV
- added U$8, U$9: TASTER9313, HeRo:TASTER9313
Connections:
- removed net PG_LEG: R19.2, R3.2, U$3.PG
- removed net PG_SERVO: R2.2, R20.2, U$4.PG
- net +3V3: no longer R2.1, R3.1
- net +5V: no longer U$1.VIN
- net GND: now also U$8.P, U$8.P1, U$9.P, U$9.P1; no longer S1.P, S1.P1, S2.P, S2.P1, U$1.GND
- net IMU_INT: no longer R21.1
- net IO17: no longer R21.2
- net IO18: no longer R19.1
- net IO19: no longer R20.1
- net N$13: now also U$8.S; no longer S1.S, S1.S1
- net N$14: now also U$9.S1; no longer S2.S, S2.S1
- net SCL_5V: no longer U$1.SCL
- net SDA_5V: no longer U$1.SDA
