File: PCB/Mainboard/Mainboard.sch (EAGLE design)
At the start: 61 parts, among them IC1 FT232RL, T1 BC847, T2 BC847

Commit message: finalised routing, added 3D-Models
Parts:
- removed IC1: FT232RL, ftdichip:FT232RL
- removed LED1, LED2, LED3, LED4, LED5, LED6, LED7: (no value), led:LEDCHIP-LED0805
- removed S3, S4, S5: (no value), switch:255SB
- removed SJ1: (no value), jumper:SJ
- removed U$2: ESP32-WROOM-32U, HeRo:ESP32-WROOM-32U
- removed U$5: BLUEDOT-BNO055, HeRo:BLUEDOT-BNO055
- removed U$7: PCA9306, HeRo:PCA9306
- added 12V, 3.3V, 5V, 6V, ESP, RX, TX: (no value), led:LEDCHIP-LED0805
- added 9-AXIS-IMU: BLUEDOT-BNO055, HeRo:BLUEDOT-BNO055
- added ESP-PWR, LEG-PWR, SERVO-PWR: CSS-1202, HeRo:CSS-1202
- added ESP32-WROOM32U: ESP32-WROOM-32U, HeRo:ESP32-WROOM-32U
- added FTDI: FT232RL, ftdichip:FT232RL
- added IMU-ADDR: (no value), jumper:SJ
- added LVL-SHIFT: PCA9306, HeRo:PCA9306
- renumbered U$3 to D24V10F5, U$4 to D24V150F6, U$6 to D24V10F3, U$8 to EN, U$9 to IO0
Connections:
- net !CTS: now also FTDI.!CTS; no longer IC1.!CTS
- net !DTR: now also FTDI.!DTR; no longer IC1.!DTR
- net !RTS: now also FTDI.!RTS; no longer IC1.!RTS
- net +3V3: now also ESP32-WROOM32U.3V3, FTDI.VCCIO, LVL-SHIFT.VREF1; no longer IC1.VCCIO, U$2.3V3, U$7.VREF1
- net +5V: now also 9-AXIS-IMU.VCC; no longer U$5.VCC
- net CLK: now also ESP32-WROOM32U.CLK; no longer U$2.CLK
- net CMD: now also ESP32-WROOM32U.CMD; no longer U$2.CMD
- net EN: now also ESP32-WROOM32U.EN; no longer U$2.EN
- net EN_3V3: now also ESP-PWR.P; no longer S5.P
- net EN_5V: now also LEG-PWR.P; no longer S4.P
- net EN_SERVO: now also SERVO-PWR.P; no longer S3.P
- net GND: now also 12V.C, 3.3V.C, 5V.C, 6V.C, 9-AXIS-IMU.GND, ESP-PWR.S, ESP.C, ESP32-WROOM32U.GND, FTDI.GND, FTDI.GND@1, FTDI.GND@2, FTDI.GND@A, FTDI.TEST, IMU-ADDR.2, LEG-PWR.S, LVL-SHIFT.GND, SERVO-PWR.S; no longer IC1.GND, IC1.GND@1, IC1.GND@2, IC1.GND@A, IC1.TEST, LED3.C, LED4.C, LED5.C, LED6.C, LED7.C, S3.S, S4.S, S5.S, SJ1.2, U$2.GND, U$5.GND, U$7.GND
- net IMU_ADR: now also 9-AXIS-IMU.ADR, IMU-ADDR.1; no longer SJ1.1, U$5.ADR
- net IMU_INT: now also 9-AXIS-IMU.INT; no longer U$5.INT
- net IO0: now also ESP32-WROOM32U.IO0; no longer U$2.IO0
- net IO12: now also ESP32-WROOM32U.IO12; no longer U$2.IO12
- net IO13: now also ESP32-WROOM32U.IO13; no longer U$2.IO13
- net IO14: now also ESP32-WROOM32U.IO14; no longer U$2.IO14
- net IO15: now also ESP32-WROOM32U.IO15; no longer U$2.IO15
- net IO16: now also ESP32-WROOM32U.IO16; no longer U$2.IO16
- net IO17: now also ESP32-WROOM32U.IO17; no longer U$2.IO17
- net IO18: now also ESP32-WROOM32U.IO18; no longer U$2.IO18
- net IO19: now also ESP32-WROOM32U.IO19; no longer U$2.IO19
- net IO2: now also ESP32-WROOM32U.IO2; no longer U$2.IO2
- net IO21: now also ESP32-WROOM32U.IO21; no longer U$2.IO21
- net IO22: now also ESP32-WROOM32U.IO22; no longer U$2.IO22
- net IO23: now also ESP32-WROOM32U.IO23; no longer U$2.IO23
- net IO25: now also ESP32-WROOM32U.IO25; no longer U$2.IO25
- net IO26: now also ESP32-WROOM32U.IO26; no longer U$2.IO26
- net IO27: now also ESP32-WROOM32U.IO27; no longer U$2.IO27
- net IO32: now also ESP32-WROOM32U.IO32; no longer U$2.IO32
- net IO33: now also ESP32-WROOM32U.IO33; no longer U$2.IO33
- net IO34: now also ESP32-WROOM32U.IO34; no longer U$2.IO34
- net IO35: now also ESP32-WROOM32U.IO35; no longer U$2.IO35
- net IO4: now also ESP32-WROOM32U.IO4; no longer U$2.IO4
- net IO5: now also ESP32-WROOM32U.IO5; no longer U$2.IO5
- net N$12: now also ESP.A; no longer LED3.A
- net N$15: now also 5V.A; no longer LED5.A
- net N$16: now also 6V.A; no longer LED6.A
- net N$17: now also 3.3V.A; no longer LED4.A
- net N$18: now also 12V.A; no longer LED7.A
- net N$23: now also LVL-SHIFT.EN, LVL-SHIFT.VREF2; no longer U$7.EN, U$7.VREF2
- net N$3: now also FTDI.!RESET; no longer IC1.!RESET
- net N$4: now also FTDI.CBUS0, TX.C; no longer IC1.CBUS0, LED1.C
- net N$5: now also FTDI.CBUS1, RX.C; no longer IC1.CBUS1, LED2.C
- net N$6: now also TX.A; no longer LED1.A
- net N$7: now also RX.A; no longer LED2.A
- net RXD: now also FTDI.RXD; no longer IC1.RXD
- net RXD0: now also ESP32-WROOM32U.RXD0; no longer U$2.RXD0
- net SCL_3V3: now also LVL-SHIFT.SCL1; no longer U$7.SCL1
- net SCL_5V: now also 9-AXIS-IMU.SCL, LVL-SHIFT.SCL2; no longer U$5.SCL, U$7.SCL2
- net SD0: now also ESP32-WROOM32U.SD0; no longer U$2.SD0
- net SD1: now also ESP32-WROOM32U.SD1; no longer U$2.SD1
- net SD2: now also ESP32-WROOM32U.SD2; no longer U$2.SD2
- net SD3: now also ESP32-WROOM32U.SD3; no longer U$2.SD3
- net SDA_3V3: now also LVL-SHIFT.SDA1; no longer U$7.SDA1
- net SDA_5V: now also 9-AXIS-IMU.SDA, LVL-SHIFT.SDA2; no longer U$5.SDA, U$7.SDA2
- net SN: now also ESP32-WROOM32U.SENSOR_VN; no longer U$2.SENSOR_VN
- net SP: now also ESP32-WROOM32U.SENSOR_VP; no longer U$2.SENSOR_VP
- net TXD: now also FTDI.TXD; no longer IC1.TXD
- net TXD0: now also ESP32-WROOM32U.TXD0; no longer U$2.TXD0
- net USB_D_N: now also FTDI.USBDM; no longer IC1.USBDM
- net USB_D_P: now also FTDI.USBDP; no longer IC1.USBDP
- net VBUS: now also FTDI.VCC; no longer IC1.VCC
